File: kicad/augmented.kicad_pcb (KiCad board)
At the start: 2 copper layers, 335.8 x 100 mm, 167 parts, among them J2 Conn_01x04, J3 Conn_01x07, J4 Conn_01x07, SW1 RESET, SW2 BOOT, U2 RP2040, U5 W25Q128JVS, Y1 12MHz

Commit message: feat: add daughterboard pcb
Parts:
- added C16: 100uF, Capacitor_SMD:C_0603_1608Metric, F.Cu at (235.3, 187.6)
- added C19: 10uF, Capacitor_SMD:C_0603_1608Metric, F.Cu at (225.3, 199.0)
- added C20: 10uF, Capacitor_SMD:C_0603_1608Metric, F.Cu at (209.7, 188.0)
- added C21: 10uF, Capacitor_SMD:C_0603_1608Metric, F.Cu at (217.7, 201.6)
- added C23: 100nF, Capacitor_SMD:C_0603_1608Metric, F.Cu at (184.3, 184.5)
- added C24: 10uF, Capacitor_SMD:C_0603_1608Metric, F.Cu at (188.7, 186.8)
- added C25: 10uF, Capacitor_SMD:C_0603_1608Metric, F.Cu at (183.5, 193.4)
- added C3: 100uF, Capacitor_SMD:C_0603_1608Metric, F.Cu at (212.6, 189.6)
- added D1: RED, LED_SMD:LED_miniPLCC_2315_Handsoldering, B.Cu at (367.2, 161.1)
- added D2: WHITE, LED_SMD:LED_miniPLCC_2315_Handsoldering, F.Cu at (106.6, 122.3)
- added D73: GREEN, LED_THT:LED_D3.0mm_Horizontal_O1.27mm_Z6.0mm, B.Cu at (191.2, 174.8)
- added D74: RED, LED_THT:LED_D3.0mm_Horizontal_O1.27mm_Z6.0mm, B.Cu at (196.3, 174.8)
- added J5: USB_A, Connector_USB:USB_A_Receptacle_XKB_U231-091N-4BLRA00-S, F.Cu at (211.1, 178.7)
- added J6: USB_A, Connector_USB:USB_A_Receptacle_XKB_U231-091N-4BLRA00-S, F.Cu at (231.1, 178.7)
- added J7: USB_C_Receptacle_USB2.0_14P, Connector_USB:USB_C_Receptacle_XKB_U262-16XN-4BVC11, F.Cu at (182.8, 175.3)
- added J8: Conn_01x04, Connector_JST:JST_GH_SM04B-GHS-TB_1x04-1MP_P1.25mm_Horizontal, F.Cu at (194.8, 180.9)
- added R10: 47k, Resistor_SMD:R_0603_1608Metric, F.Cu at (211.9, 201.1)
- added R11: 100k, Resistor_SMD:R_0603_1608Metric, F.Cu at (211.7, 195.0)
- added R12: 2.7k, Resistor_SMD:R_0603_1608Metric, F.Cu at (216.7, 188.8)
- added R13: 330, Resistor_SMD:R_0603_1608Metric, F.Cu at (201.8, 177.6)
- added R14: 330, Resistor_SMD:R_0603_1608Metric, F.Cu at (201.8, 175.7)
- added R15: 5.1k, Resistor_SMD:R_0603_1608Metric, F.Cu at (184.9, 181.7)
- added R16: 5.1k, Resistor_SMD:R_0603_1608Metric, F.Cu at (180.1, 181.8)
- added R7: 1k, Resistor_SMD:R_0603_1608Metric, B.Cu at (367.1, 159.1)
- added R8: 1k, Resistor_SMD:R_0603_1608Metric, F.Cu at (109.6, 123.8)
- added R9: 100k, Resistor_SMD:R_0603_1608Metric, F.Cu at (211.9, 198.6)
- added U5: FE1.1s, Package_SO:SSOP-28_3.9x9.9mm_P0.635mm, F.Cu at (220.7, 194.6)
- added U6: USBLC6-2P6, Package_TO_SOT_SMD:SOT-666, F.Cu at (182.7, 181.8)
- added U7: NCP1117-3.3_SOT223, Package_TO_SOT_SMD:SOT-223-3_TabPin2, F.Cu at (183.2, 188.9)
- added Y2: 12MHz, Crystal:Crystal_SMD_Abracon_ABM3-2Pin_5.0x3.2mm, F.Cu at (230.9, 194.6)
- moved C10 1.11 mm to (351.5, 157.4)
- renumbered C6 to C1, C12 to C10, C16 to C11, C20 to C12, C18 to C14, C17 to C15, C7 to C2, C9 to C4, C14 to C5, C10 to C6, C15 to C7, C11 to C8, C19 to C9, D11 to D10, D12 to D11, D13 to D12, D14 to D13, D15 to D14, D16 to D15, D17 to D16, D18 to D17, D19 to D18, D20 to D19, D21 to D20, D22 to D21, D23 to D22, D24 to D23, D25 to D24, D26 to D25, D27 to D26, D28 to D27, D29 to D28, D30 to D29, D4 to D3, D31 to D30, D32 to D31, D33 to D32, D34 to D33, D35 to D34, D36 to D35, D37 to D36, D38 to D37, D39 to D38, D40 to D39, D5 to D4, D41 to D40, D42 to D41, D43 to D42, D44 to D43, D45 to D44, D46 to D45, D47 to D46, D48 to D47, D49 to D48, D50 to D49, D6 to D5, D51 to D50, D52 to D51, D53 to D52, D54 to D53, D55 to D54, D56 to D55, D57 to D56, D58 to D57, D59 to D58, D60 to D59, D7 to D6, D61 to D60, D62 to D61, D63 to D62, D64 to D63, D65 to D64, D66 to D65, D67 to D66, D68 to D67, D69 to D68, D70 to D69, D8 to D7, D71 to D70, D72 to D71, D73 to D72, D9 to D8, D10 to D9, J4 to J3, J3 to J4, MX71 to MX11, MX11 to MX12, MX12 to MX13, MX13 to MX14, MX14 to MX15, MX15 to MX16, MX16 to MX17, MX17 to MX18, MX18 to MX19, MX19 to MX20, MX20 to MX21, MX21 to MX22, MX22 to MX23, MX23 to MX24, MX24 to MX25, MX25 to MX26, MX26 to MX27, MX27 to MX28, MX28 to MX29, MX29 to MX30, MX30 to MX31, MX31 to MX32, MX32 to MX33, MX33 to MX34, MX34 to MX35, MX35 to MX36, MX36 to MX37, MX37 to MX38, MX38 to MX39, MX39 to MX40, MX40 to MX41, MX41 to MX42, MX42 to MX43, MX43 to MX44, MX44 to MX45, MX45 to MX46, MX46 to MX47, MX47 to MX48, MX48 to MX49, MX49 to MX50, MX50 to MX51, MX51 to MX52, MX52 to MX53, MX53 to MX54, MX54 to MX55, MX55 to MX56, MX56 to MX57, MX57 to MX58, MX58 to MX59, MX59 to MX60, MX60 to MX61, MX61 to MX62, MX62 to MX63, MX63 to MX64, MX64 to MX65, MX65 to MX66, MX66 to MX67, MX67 to MX68, MX68 to MX69, MX69 to MX70, MX70 to MX71, R8 to R1, R7 to R2, R11 to R3, R12 to R4, SW2 to SW1, SW1 to SW2, U2 to U1, U5 to U3
Connections:
- net /USB_D+ renamed USB_D+
- net /USB_D- renamed USB_D-
- J3 pad 1: ROW3 -> ROW4
- J3 pad 2: ROW4 -> ROW3
- J4 pad 6: ROW4 -> ROW3
- J4 pad 7: ROW3 -> ROW4
- U1 pad 29: unconnected-(U2-GPIO18-Pad29) -> /LED_CAPS
- U1 pad 9: unconnected-(U2-GPIO7-Pad9) -> /PWR_LED
Routing:
- net GND: track 118.0 -> 530.7 mm, vias 13 -> 18
- net +3V3: track 82.9 -> 392.0 mm, vias 5 -> 12
- net /LED_CAPS: track 0.00 -> 266.7 mm, vias 0 -> 3
- net +5V: track 0.00 -> 112.6 mm, vias 0 -> 4
- net (no net): track 0.00 -> 64.7 mm
- net USB_D+: track 6.47 -> 57.4 mm, vias 0 -> 1
- net Net-(D73-A): track 0.00 -> 50.8 mm, vias 0 -> 1
- net USB_D-: track 6.16 -> 51.6 mm, vias 0 -> 2
- net Net-(D74-A): track 0.00 -> 42.8 mm, vias 0 -> 1
- net Net-(J6-D-): track 0.00 -> 17.2 mm
- net ROW3: track 344.3 -> 360.4 mm
- net Net-(J6-D+): track 0.00 -> 15.8 mm
- net Net-(U5-XOUT): track 0.00 -> 13.9 mm
- net Net-(J5-D+): track 0.00 -> 13.9 mm
- net +1V8: track 0.00 -> 13.7 mm
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Other:
- board size 335.8 x 100 mm -> 335.8 x 138.7 mm
