File: kicad/daughterboard.kicad_sch (KiCad schematic)
At the start: 26 parts, among them J1 USB_C_Receptacle_USB2.0_14P, J2 Conn_01x04, J3 USB_A, J5 USB_A, U1 USBLC6-2P6, U3 NCP1117-3.3_SOT223, U4 FE1.1s, Y2 12MHz

Commit message: feat: add daughterboard pcb
Parts:
- removed C19, C20: 100uF, symbol Device:C_Polarized_Small_US
- added C16, C3: 100uF, Capacitor_SMD:C_0603_1608Metric, symbol Device:C_Small
- C19: renamed from C3; footprint Capacitor_SMD:C_0805_2012Metric -> Capacitor_SMD:C_0603_1608Metric
- C20: renamed from C4; footprint Capacitor_SMD:C_0805_2012Metric -> Capacitor_SMD:C_0603_1608Metric
- C21: renamed from C23; footprint Capacitor_SMD:C_0805_2012Metric -> Capacitor_SMD:C_0603_1608Metric
- C23: renamed from C2; footprint Capacitor_SMD:C_0805_2012Metric -> Capacitor_SMD:C_0603_1608Metric
- C24: renamed from C5; footprint Capacitor_SMD:C_0805_2012Metric -> Capacitor_SMD:C_0603_1608Metric
- C25: renamed from C8; footprint Capacitor_SMD:C_0805_2012Metric -> Capacitor_SMD:C_0603_1608Metric
- D73: renamed from D74; footprint (none) -> LED_THT:LED_D2.0mm_W4.0mm_H2.8mm_FlatTop
- D74: renamed from D1; footprint (none) -> LED_THT:LED_D2.0mm_W4.0mm_H2.8mm_FlatTop
- J5: renamed from J3; footprint (none) -> Connector_USB:USB_A_Receptacle_XKB_U231-091N-4BLRA00-S
- J6: renamed from J5; footprint (none) -> Connector_USB:USB_A_Receptacle_XKB_U231-091N-4BLRA00-S
- J7: renamed from J1; footprint (none) -> Connector_USB:USB_C_Receptacle_XKB_U262-16XN-4BVC11
- R10: renamed from R14; footprint (none) -> Resistor_SMD:R_0603_1608Metric
- R11: renamed from R10; footprint (none) -> Resistor_SMD:R_0603_1608Metric
- R12: renamed from R9; footprint (none) -> Resistor_SMD:R_0603_1608Metric
- R13: renamed from R16; footprint (none) -> Resistor_SMD:R_0603_1608Metric
- R14: renamed from R15; footprint (none) -> Resistor_SMD:R_0603_1608Metric
- R15: renamed from R3; footprint Resistor_SMD:R_0805_2012Metric -> Resistor_SMD:R_0603_1608Metric
- R16: renamed from R4; footprint Resistor_SMD:R_0805_2012Metric -> Resistor_SMD:R_0603_1608Metric
- R9: renamed from R13; footprint (none) -> Resistor_SMD:R_0603_1608Metric
- Y2: footprint (none) -> Crystal:Crystal_SMD_Abracon_ABM3-2Pin_5.0x3.2mm
- renumbered J2 to J8, U4 to U5, U1 to U6, U3 to U7
Connections:
- net USB_DM+ is gone; now on net USB_D+: U6.4 (I/O2)
- net USB_DM- is gone; now on net USB_D-: U6.6 (I/O1)
- net +5V: now also C16.1, C3.1
- net GND: now also C16.2, C3.2
