File: kicad/matrix.kicad_sch (KiCad schematic)
At the start: 141 parts

Commit message: feat: add daughterboard pcb
Parts:
- renumbered D11 to D10, D12 to D11, D13 to D12, D14 to D13, D15 to D14, D16 to D15, D17 to D16, D18 to D17, D19 to D18, D20 to D19, D21 to D20, D22 to D21, D23 to D22, D24 to D23, D25 to D24, D26 to D25, D27 to D26, D28 to D27, D29 to D28, D30 to D29, D4 to D3, D31 to D30, D32 to D31, D33 to D32, D34 to D33, D35 to D34, D36 to D35, D37 to D36, D38 to D37, D39 to D38, D40 to D39, D5 to D4, D41 to D40, D42 to D41, D43 to D42, D44 to D43, D45 to D44, D46 to D45, D47 to D46, D48 to D47, D49 to D48, D50 to D49, D6 to D5, D51 to D50, D52 to D51, D53 to D52, D54 to D53, D55 to D54, D56 to D55, D57 to D56, D58 to D57, D59 to D58, D60 to D59, D7 to D6, D61 to D60, D62 to D61, D63 to D62, D64 to D63, D65 to D64, D66 to D65, D67 to D66, D68 to D67, D69 to D68, D70 to D69, D8 to D7, D71 to D70, D72 to D71, D73 to D72, D9 to D8, D10 to D9, MX71 to MX11, MX11 to MX12, MX12 to MX13, MX13 to MX14, MX14 to MX15, MX15 to MX16, MX16 to MX17, MX17 to MX18, MX18 to MX19, MX19 to MX20, MX20 to MX21, MX21 to MX22, MX22 to MX23, MX23 to MX24, MX24 to MX25, MX25 to MX26, MX26 to MX27, MX27 to MX28, MX28 to MX29, MX29 to MX30, MX30 to MX31, MX31 to MX32, MX32 to MX33, MX33 to MX34, MX34 to MX35, MX35 to MX36, MX36 to MX37, MX37 to MX38, MX38 to MX39, MX39 to MX40, MX40 to MX41, MX41 to MX42, MX42 to MX43, MX43 to MX44, MX44 to MX45, MX45 to MX46, MX46 to MX47, MX47 to MX48, MX48 to MX49, MX49 to MX50, MX50 to MX51, MX51 to MX52, MX52 to MX53, MX53 to MX54, MX54 to MX55, MX55 to MX56, MX56 to MX57, MX57 to MX58, MX58 to MX59, MX59 to MX60, MX60 to MX61, MX61 to MX62, MX62 to MX63, MX63 to MX64, MX64 to MX65, MX65 to MX66, MX66 to MX67, MX67 to MX68, MX68 to MX69, MX69 to MX70, MX70 to MX71
